File: mouse_hardware.kicad_sch (KiCad schematic)
At the start: 7 parts, among them U1 TPS73601DBV

Commit message: Start pcb schematic
Parts:
- added C5, C6, C7, C8: C, symbol Device:C
- added R3, R4, R6: R, symbol Device:R
- added R5: 56K, symbol Device:R
- added U2: TPS73601DBV, Package_TO_SOT_SMD:SOT-23-5, symbol Regulator_Linear:TPS73601DBV
Connections:
- net +5V: now also C5.1, C6.1, U2.1 (IN), U2.3 (EN)
- net GND: now also C5.2, C6.2, C8.2, R5.1, U2.2 (GND)
- net at C3.1, C4.1, R2.2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: now also R3.2
- new net: C7.1, C8.1, R4.2, R6.2, U2.5 (OUT)
- new net: C7.2, R4.1, R5.2, U2.4 (FB)
- new net +3.3V: R3.1
Other:
- moved on the sheet: C1, C2, C3, C4, R1, R2, U1

Commit message: Start designing pcb
Parts:
- removed R3, R4, R6: R, symbol Device:R
- removed R5: 56K, symbol Device:R
- removed U1, U2: TPS73601DBV, Package_TO_SOT_SMD:SOT-23-5, symbol Regulator_Linear:TPS73601DBV
- added C10, C11, C12, C9: 1uF, symbol Device:C
- added IC1: ADP150AUJZ-2.0-R7, SOT95P280X100-5N, symbol ADP150AUJZ:ADP150AUJZ-2.0-R7
- added IC2: AP2112K-3.3TRG1, SOT95P282X130-5N, symbol AP2112K-3:AP2112K-3.3TRG1
- added U1: STM32F103RETx, Package_QFP:LQFP-64_10x10mm_P0.5mm, symbol MCU_ST_STM32F1:STM32F103RETx
- C1: value C -> 1uF
- C2: value C -> 10nF
- C3, C5, C6, C7, C8: value C -> 100nF
- C4: value C -> 4.7uF
- R2: value R -> 10K
Connections:
- net +5V: now also C11.2, C9.2, IC1.1 (VIN), IC1.3 (EN), IC2.1 (VIN), IC2.3 (EN); no longer C1.1, C2.1, C5.1, C6.1
- net GND: now also C3.2, C7.2, R2.2, C10.1, C11.1, C12.1, C9.1, IC1.2 (GND), IC2.2 (GND), U1.12 (VSSA), U1.18 (VSS), U1.31 (VSS), U1.47 (VSS), U1.63 (VSS)
- net +3V3: now reaches C7.1, C8.1
- net +3V3: now also C1.1, C2.1, C3.1, C4.1, C5.1, C6.1, C12.2, IC2.5 (VOUT), U1.1 (VBAT), U1.13 (VDDA), U1.19 (VDD), U1.32 (VDD), U1.48 (VDD), U1.64 (VDD)
- new net: R2.1, U1.28 (PB2)
- new net: R1.2, U1.60 (BOOT0)
- new net +2V: C10.2, IC1.5 (VOUT)
- new net NRST: U1.7 (NRST)
- new net USBDM: U1.30 (PB11)
- no-connect marks 0 -> 1

Commit message: Start designing pcb
Parts:
- added Y1: LFXTAL029914Reel, LFXTAL029914Reel, symbol LFXTAL029914:LFXTAL029914Reel
Changed lines of the file:
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@@
+    (stroke (width 0) (type default))
+  )
+  (wire (pts (xy 133.35 102.87) (xy 129.54 102.87))
     (stroke (width 0) (type default))
   )
@@
   )
   (wire (pts (xy 30.48 57.15) (xy 30.48 58.42))
+    (stroke (width 0) (type default))
+  )
+  (wire (pts (xy 129.54 102.87) (xy 129.54 106.68))
     (stroke (width 0) (type default))
   )
@@
         )
       )
+    )
+  )
+  (symbol (lib_id "LFXTAL029914:LFXTAL029914Reel") (at 133.35 102.87 0) (unit 1)
+    (in_bom yes) (on_board yes) (dnp no) (fields_autoplaced)
+    (property "Reference" "Y1" (at 138.43 93.98 0)
+      (effects (font (size 1.27 1.27)))
+    )
+    (property "Value" "LFXTAL029914Reel" (at 138.43 96.52 0)
+      (effects (font (size 1.27 1.27)))
+    )
+    (property "Footprint" "LFXTAL029914Reel" (at 142.24 199.06 0)
+      (effects (font (size 1.27 1.27)) (justify left top) hide)
+    )
+    (property "Datasheet" "https://datasheet.datasheetarchive.com/originals/dk/DKDS-40/46251.pdf" (at 142.24 299.06 0)
+      (effects (font (size 1.27 1.27)) (justify left top) hide)
+    )
+    (property "Height" "4.3" (at 142.24 499.06 0)
+      (effects (font (size 1.27 1.27)) (justify left top) hide)
+    )
+    (property "Mouser Part Number" "449-LFXTAL029914REEL" (at 142.24 599.06 0)
+      (effects (font (size 1.27 1.27)) (justify left top) hide)
+    )
+    (property "Mouser Price/Stock" "https://www.mouser.co.uk/ProductDetail/IQD/LFXTAL029914Reel?qs=e4%2FAndAAwgJ9bR%252BzpdWpUQ%3D%3D" (at 142.24 699.06 0)
+      (effects (font (size 1.27 1.27)) (justify left top) hide)
+    )
+    (property "Manufacturer_Name" "IQD" (at 142.24 799.06 0)
+      (effects (font (size 1.27 1.27)) (justify left top) hide)
+    )
+    (property "Manufacturer_Part_Number" "LFXTAL029914Reel" (at 142.24 899.06 0)
+      (effects (font (size 1.27 1.27)) (justify left top) hide)
+    )
+    (pin "")
+    (pin "2")
+    (instances
+      (project "mouse_hardware"
+        (path "/0578f8d8-597b-427f-bd65-a1426fa348f5"
+          (reference "Y1") (unit 1)
+        )
+      )

Commit message: Start designing pcb
Parts:
- added C13, C14, C15, C16, C17, C18: 100nF, symbol Device:C
- added R3: R, symbol Device:R
- added R4, R5, R6, R7: 10K, symbol Device:R
- added SW1: SW_Push, symbol Switch:SW_Push
- added SW2, SW3, SW4, SW5: SW_DPDT_x2, symbol Switch:SW_DPDT_x2
- added U2: PMW3360DM-T2QU, symbol PMW3360:PMW3360DM-T2QU
Connections:
- net +3V3: now also R3.2, R4.1, R5.1, R6.1, R7.1
- net GND: now also C13.2, C14.2, C15.2, C16.2, C17.2, C18.2, SW1.2, SW2.3 (C), SW3.3 (C), SW4.3 (C), SW5.3 (C)
- net NRST: now also R3.1, SW1.1
- net OSC_OUT: now reaches Y1.
- net OSC_OUT: now also C18.1
- net OSC_IN: now reaches Y1.2 (X2)
- net OSC_IN: now also C17.1
- new net DPI_SWITCH: C16.1, R7.2, SW5.1 (A), SW5.2 (B)
- new net LEFT_CLICK: C13.1, R4.2, SW2.1 (A), SW2.2 (B)
- new net MIDDLE_CLICK: C15.1, R6.2, SW4.1 (A), SW4.2 (B)
- new net RIGHT_CLICK: C14.1, R5.2, SW3.1 (A), SW3.2 (B)

Commit message: Start designing pcb
Parts:
- added C19, C20: C, Capacitor_SMD:C_0805_2012Metric_Pad1.18x1.45mm_HandSolder, symbol Device:C
- added D1, D2: LED, LED_SMD:LED_0805_2012Metric_Pad1.15x1.40mm_HandSolder, symbol Device:LED
- added J1: Conn_01x04_Pin, Connector_PinHeader_2.54mm:PinHeader_1x04_P2.54mm_Horizontal, symbol Connector:Conn_01x04_Pin
- added R10, R9: 70R, Resistor_SMD:R_0805_2012Metric_Pad1.20x1.40mm_HandSolder, symbol Device:R
- added R8: R, Resistor_SMD:R_0805_2012Metric_Pad1.20x1.40mm_HandSolder, symbol Device:R
- C1, C10, C11, C12, C13, C14, C15, C16, C2, C3, C4, C5, C6, C7, C8, C9: footprint (none) -> Capacitor_SMD:C_0805_2012Metric_Pad1.18x1.45mm_HandSolder
- C17, C18: value 100nF -> 16pF; footprint (none) -> Capacitor_SMD:C_0805_2012Metric_Pad1.18x1.45mm_HandSolder
- R1: value R -> 10k; footprint (none) -> Resistor_SMD:R_0805_2012Metric_Pad1.20x1.40mm_HandSolder
- R2, R3, R4, R5, R6, R7: footprint (none) -> Resistor_SMD:R_0805_2012Metric_Pad1.20x1.40mm_HandSolder
Connections:
- net +2V: now also U2.15 (LED_P), U2.4 (VDD)
- net +3V3: now also U2.5 (VDDIO), D2.2 (A), R8.1
- net +5V: now also J1.1 (Pin_1)
- net GND: now also U2.8 (GND), C19.2, C20.2, J1.4 (Pin_4), R10.2, R9.2
- net NRST: now also U2.7 (~{RESET})
- net USBDM: now also J1.3 (Pin_3)
- net USBDP: now also U1.33 (PB12), J1.2 (Pin_2)
- net SCK: now reaches U2.10 (SCLK)
- net SCK: now also U1.21 (PA5)
- net MOSI: now reaches U2.11 (MOSI)
- net MOSI: now also U1.23 (PA7)
- net MISO: now reaches U2.12 (MISO)
- net MISO: now also U1.22 (PA6), R8.2
- net NCS: now reaches U2.13 (~{CS})
- net NCS: now also U1.20 (PA4)
- net at U2.3 (VDDPIX): now also C19.1, C20.1
- net MOTION: now reaches U2.9 (MOTION)
- net MOTION: now also U1.26 (PB0)
- net STATUS_LED: now reaches U1.14 (PA0)
- net STATUS_LED: now also D1.2 (A)
- new net: D2.1 (K), R10.1
- new net: D1.1 (K), R9.1

Commit message: Finish making schematic
Parts:
- removed SW2, SW3, SW4, SW5: SW_DPDT_x2, symbol Switch:SW_DPDT_x2
- removed Y1: LFXTAL029914Reel, LFXTAL029914Reel, symbol LFXTAL029914:LFXTAL029914Reel
- added R11: 39R, Resistor_SMD:R_0805_2012Metric_Pad1.20x1.40mm_HandSolder, symbol Device:R
- added S1, S2, S3: D2F-FL, D2FFL, symbol D2F-FL:D2F-FL
- added SW5: SW_Push, 147873-1:1478731, symbol Switch:SW_Push
- added Y1: 8MHz, Crystal:Crystal_SMD_HC49-SD_HandSoldering, symbol Device:Crystal
- C17, C18: value 16pF -> 20pF
- C19: value C -> 100nF
- C20: value C -> 4.7uF
- R8: value R -> 10K
- SW1: footprint (none) -> 147873-1:1478731
- U2: footprint (none) -> PMW3360DM:PMW3360
Connections:
- net +2V: now also R11.1; no longer U2.15 (LED_P)
- net DPI_SWITCH: now also SW5.1
- net GND: now also S1.1 (COM), S2.1 (COM), S3.1 (COM), SW5.2
- net LEFT_CLICK: now also S1.2 (NO)
- net MIDDLE_CLICK: now also S3.2 (NO)
- net OSC_IN: now also Y1.1
- net OSC_OUT: now also Y1.2
- net RIGHT_CLICK: now also S2.2 (NO)
- new net: R11.2, U2.15 (LED_P)
- no-connect marks 1 -> 43
Other:
- moved on the sheet: C13, R4

Commit message: Start routing
Parts:
- added J2: Conn_01x04_Pin, Connector_PinHeader_2.54mm:PinHeader_1x04_P2.54mm_Horizontal, symbol Connector:Conn_01x04_Pin
- R3: value R -> 10K
Connections:
- net +5V: now also J2.1 (Pin_1)
- net GND: now also J2.4 (Pin_4)
- net OSC_IN: now also U1.5 (PD0)
- net OSC_OUT: now also U1.6 (PD1)
- new net SWCLK: J2.3 (Pin_3)
- new net SWDIO: J2.2 (Pin_2)
- no-connect marks 43 -> 41
Changed lines of the file:
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@@
   (no_connect (at 191.77 162.56))
   (no_connect (at 191.77 144.78))
-  (no_connect (at 191.77 137.16))
   (no_connect (at 191.77 165.1))
   (no_connect (at 191.77 149.86))
@@
   (no_connect (at 191.77 170.18))
   (no_connect (at 191.77 157.48))
-  (no_connect (at 191.77 134.62))
   (no_connect (at 191.77 152.4))
   (no_connect (at 227.33 152.4))
@@
     (stroke (width 0) (type default))
   )
+  (wire (pts (xy 287.655 170.815) (xy 289.56 170.815))
+    (stroke (width 0) (type default))
+  )
   (wire (pts (xy 85.09 58.42) (xy 85.09 59.69))
     (stroke (width 0) (type default))
@@
     (stroke (width 0) (type default))
   )
+  (wire (pts (xy 287.655 163.195) (xy 290.195 163.195))
+    (stroke (width 0) (type default))
+  )
   (wire (pts (xy 285.75 66.04) (xy 283.21 66.04))
     (stroke (width 0) (type default))
@@
   )
   (wire (pts (xy 77.47 30.48) (xy 82.55 30.48))
+    (stroke (width 0) (type default))
+  )
+  (wire (pts (xy 289.56 170.815) (xy 289.56 172.085))
     (stroke (width 0) (type default))
   )
@@
     )
   )
+  (global_label "SWCLK" (shape input) (at 287.655 168.275 0) (fields_autoplaced)
+    (effects (font (size 1.27 1.27)) (justify left))
+    (property "Intersheetrefs" "${INTERSHEET_REFS}" (at 296.8692 168.275 0)
+      (effects (font (size 1.27 1.27)) (justify left) hide)
+    )
+  )
   (global_label "OSC_IN" (shape input) (at 127 102.87 180) (fields_autoplaced)
     (effects (font (size 1.27 1.27)) (justify right))
@@
     )
   )
+  (global_label "SWDIO" (shape input) (at 287.655 165.735 0) (fields_autoplaced)
+    (effects (font (size 1.27 1.27)) (justify left))
+    (property "Intersheetrefs" "${INTERSHEET_REFS}" (at 296.5064 165.735 0)
+      (effects (font (size 1.27 1.27)) (justify left) hide)
+    )
+  )
   (global_label "LEFT_CLICK" (shape input) (at 101.6 180.34 0) (fields_autoplaced)
     (effects (font (size 1.27 1.27)) (justify left))
@@
     )
   )
+  (global_label "OSC_OUT" (shape input) (at 191.77 137.16 180) (fields_autoplaced)
+    (effects (font (size 1.27 1.27)) (justify right))
+    (property "Intersheetrefs" "${INTERSHEET_REFS}" (at 180.3786 137.16 0)
+      (effects (font (size 1.27 1.27)) (justify right) hide)
+    )
+  )
   (global_label "NRST" (shape input) (at 77.47 93.98 180) (fields_autoplaced)
     (effects (font (size 1 1)) (justify right))
@@
     )
   )
+  (global_label "OSC_IN" (shape input) (at 191.77 134.62 180) (fields_autoplaced)
+    (effects (font (size 1.27 1.27)) (justify right))
+    (property "Intersheetrefs" "${INTERSHEET_REFS}" (at 182.0719 134.62 0)
+      (effects (font (size 1.27 1.27)) (justify right) hide)
+    )
+  )
   (global_label "RIGHT_CLICK" (shape input) (at 100.33 214.63 0) (fields_autoplaced)
     (effects (font (size 1.27 1.27)) (justify left))
@@
     )
   )
+  (symbol (lib_id "power:+5V") (at 290.195 163.195 270) (unit 1)
+    (in_bom yes) (on_board yes) (dnp no) (fields_autoplaced)
+    (property "Reference" "#PWR046" (at 286.385 163.195 0)
+      (effects (font (size 1.27 1.27)) hide)
+    )
+    (property "Value" "+5V" (at 294.005 163.195 90)
+      (effects (font (size 1.27 1.27)) (justify left))
+    )
+    (property "Footprint" "" (at 290.195 163.195 0)
+      (effects (font (size 1.27 1.27)) hide)
+    )
+    (property "Datasheet" "" (at 290.195 163.195 0)
+      (effects (font (size 1.27 1.27)) hide)
+    )
+    (pin "1")
+    (instances
+      (project "mouse_hardware"
+        (path "/0578f8d8-597b-427f-bd65-a1426fa348f5"
+          (reference "#PWR046") (unit 1)
+        )
+      )
+    )
+  )
   (symbol (lib_id "power:+3V3") (at 278.13 60.96 90) (unit 1)
     (in_bom yes) (on_board yes) (dnp no) (fields_autoplaced)
@@
         (path "/0578f8d8-597b-427f-bd65-a1426fa348f5"
           (reference "#PWR05") (unit 1)
+        )
+      )
+    )
+  )
+  (symbol (lib_id "power:GND") (at 289.56 172.085 0) (unit 1)
+    (in_bom yes) (on_board yes) (dnp no) (fields_autoplaced)
+    (property "Reference" "#PWR047" (at 289.56 178.435 0)
+      (effects (font (size 1.27 1.27)) hide)
+    )
+    (property "Value" "GND" (at 289.56 177.165 0)
+      (effects (font (size 1.27 1.27)))
+    )
+    (property "Footprint" "" (at 289.56 172.085 0)
+      (effects (font (size 1.27 1.27)) hide)
+    )
+    (property "Datasheet" "" (at 289.56 172.085 0)
+      (effects (font (size 1.27 1.27)) hide)
+    )
+    (pin "1")
+    (instances
+      (project "mouse_hardware"
+        (path "/0578f8d8-597b-427f-bd65-a1426fa348f5"
+          (reference "#PWR047") (unit 1)
         )
       )
@@
       (effects (font (size 1.27 1.27)))
     )
-    (property "Value" "R" (at 78.74 87.63 90)
+    (property "Value" "10K" (at 78.74 87.63 90)
       (effects (font (size 1.27 1.27)))
     )
@@
         )
       )
+    )
+  )
+  (symbol (lib_id "Connector:Conn_01x04_Pin") (at 282.575 165.735 0) (unit 1)
+    (in_bom yes) (on_board yes) (dnp no) (fields_autoplaced)
+    (property "Reference" "J2" (at 283.21 158.115 0)
+      (effects (font (size 1.27 1.27)))
+    )
+    (property "Value" "Conn_01x04_Pin" (at 283.21 160.655 0)
+      (effects (font (size 1.27 1.27)))
+    )
+    (property "Footprint" "Connector_PinHeader_2.54mm:PinHeader_1x04_P2.54mm_Horizontal" (at 282.575 165.735 0)
+      (effects (font (size 1.27 1.27)) hide)
+    )
+    (property "Datasheet" "~" (at 282.575 165.735 0)
+      (effects (font (size 1.27 1.27)) hide)
+    )
+    (pin "1")
+    (pin "2")
+    (pin "3")
+    (pin "4")
+    (instances
+      (project "mouse_hardware"
+        (path "/0578f8d8-597b-427f-bd65-a1426fa348f5"
+          (reference "J2") (unit 1)
+        )
+      )

Commit message: Finish designing and routing pcb
Parts:
- added H1, H2, H3: MountingHole_Pad, symbol Mechanical:MountingHole_Pad
Changed lines of the file:
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@@
+    )
+  )
+  (symbol (lib_id "Mechanical:MountingHole_Pad") (at 44.45 180.34 0) (unit 1)
+    (in_bom yes) (on_board yes) (dnp no) (fields_autoplaced)
+    (property "Reference" "H1" (at 46.99 177.8 0)
+      (effects (font (size 1.27 1.27)) (justify left))
+    )
+    (property "Value" "MountingHole_Pad" (at 46.99 180.34 0)
+      (effects (font (size 1.27 1.27)) (justify left))
+    )
+    (property "Footprint" "" (at 44.45 180.34 0)
+      (effects (font (size 1.27 1.27)) hide)
+    )
+    (property "Datasheet" "~" (at 44.45 180.34 0)
+      (effects (font (size 1.27 1.27)) hide)
+    )
+    (pin "1")
+    (instances
+      (project "mouse_hardware"
+        (path "/0578f8d8-597b-427f-bd65-a1426fa348f5"
+          (reference "H1") (unit 1)
+        )
+      )
     )
   )
@@
     )
   )
+  (symbol (lib_id "Mechanical:MountingHole_Pad") (at 41.91 214.63 0) (unit 1)
+    (in_bom yes) (on_board yes) (dnp no) (fields_autoplaced)
+    (property "Reference" "H2" (at 44.45 212.09 0)
+      (effects (font (size 1.27 1.27)) (justify left))
+    )
+    (property "Value" "MountingHole_Pad" (at 44.45 214.63 0)
+      (effects (font (size 1.27 1.27)) (justify left))
+    )
+    (property "Footprint" "" (at 41.91 214.63 0)
+      (effects (font (size 1.27 1.27)) hide)
+    )
+    (property "Datasheet" "~" (at 41.91 214.63 0)
+      (effects (font (size 1.27 1.27)) hide)
+    )
+    (pin "1")
+    (instances
+      (project "mouse_hardware"
+        (path "/0578f8d8-597b-427f-bd65-a1426fa348f5"
+          (reference "H2") (unit 1)
+        )
+      )
+    )
+  )
   (symbol (lib_id "D2F-FL:D2F-FL") (at 82.55 217.17 180) (unit 1)
     (in_bom yes) (on_board yes) (dnp no) (fields_autoplaced)
@@
         )
       )
+    )
+  )
+  (symbol (lib_id "Mechanical:MountingHole_Pad") (at 41.275 251.46 0) (unit 1)
+    (in_bom yes) (on_board yes) (dnp no) (fields_autoplaced)
+    (property "Reference" "H3" (at 43.815 248.92 0)
+      (effects (font (size 1.27 1.27)) (justify left))
+    )
+    (property "Value" "MountingHole_Pad" (at 43.815 251.46 0)
+      (effects (font (size 1.27 1.27)) (justify left))
+    )
+    (property "Footprint" "" (at 41.275 251.46 0)
+      (effects (font (size 1.27 1.27)) hide)
+    )
+    (property "Datasheet" "~" (at 41.275 251.46 0)
+      (effects (font (size 1.27 1.27)) hide)
+    )
+    (pin "1")
+    (instances
+      (project "mouse_hardware"
+        (path "/0578f8d8-597b-427f-bd65-a1426fa348f5"
+          (reference "H3") (unit 1)
+        )
+      )
