File: mouse_hardware.kicad_pcb (KiCad board)
At the start: 4 copper layers, 51 x 82 mm, 48 parts, among them IC1 ADP150AUJZ-2.0-R7, IC2 AP2112K-3.3TRG1, J1 Conn_01x04_Pin, J2 Conn_01x04_Pin, SW1 SW_Push, SW5 SW_Push, U1 STM32F103RETx, U2 PMW3360DM-T2QU, Y1 8MHz

Commit message: Re-reference and update pcb from schematic
Parts:
- removed the C16 at (20.5, 65.2)
- removed the R7 at (17.0, 65.3)
- removed SW5: SW_Push, 147873-1:1478731
- added C3: 100nF, Capacitor_SMD:C_0805_2012Metric_Pad1.18x1.45mm_HandSolder, F.Cu at (21.5, 63.0)
- added C4: 100nF, Capacitor_SMD:C_0805_2012Metric_Pad1.18x1.45mm_HandSolder, F.Cu at (21.5, 66.0)
- added R2: 10K, Resistor_SMD:R_0805_2012Metric_Pad1.20x1.40mm_HandSolder, F.Cu at (21.5, 68.5)
- added SW2: SW_Push, 147873-1:1478731, F.Cu at (20.5, 56.0)
- renumbered C9 to C1, C17 to C10, C18 to C11, C8 to C12, C7 to C13, C5 to C14, C6 to C15, C3 to C16, C4 to C17, C2 to C18, C1 to C19, C11 to C2, C19 to C21, C10 to C5, C12 to C6, C15 to C7, C14 to C8, C13 to C9, H3 to H1, H1 to H3, R3 to R1, R11 to R10, R8 to R11, R6 to R3, R5 to R4, R4 to R5, R9 to R6, R10 to R7, R1 to R8, R2 to R9, S3 to S1, S1 to S3
Connections:
- U1 pad 10: unconnected-(U1-PC2-Pad10) -> DPI_SWITCH
- U1 pad 11: unconnected-(U1-PC3-Pad11) -> LEFT_CLICK
- U1 pad 14: STATUS_LED -> unconnected-(U1-PA0-Pad14)
- U1 pad 24: unconnected-(U1-PC4-Pad24) -> RIGHT_CLICK
- U1 pad 25: unconnected-(U1-PC5-Pad25) -> MIDDLE_CLICK
- U1 pad 26: MOTION -> unconnected-(U1-PB0-Pad26)
- U1 pad 8: unconnected-(U1-PC0-Pad8) -> STATUS_LED
- U1 pad 9: unconnected-(U1-PC1-Pad9) -> MOTION
Routing:
- net DPI_SWITCH: track 12.8 -> 0.00 mm
- net +3V3: track 106.2 -> 102.2 mm, vias 26 -> 24

Commit message: Start re-routing
Parts:
- moved R11 9.20 mm to (50.0, 61.5), turned to 180 degrees
- moved C18 2.26 mm to (47.0, 76.5), turned to 90 degrees
- moved C19 1.96 mm to (45.8, 73.1), turned to 180 degrees
- moved R1 0.86 mm to (28.5, 77.0)
Routing:
- net STATUS_LED: track 108.2 -> 0.00 mm, vias 4 -> 0
- net +5V: track 101.1 -> 14.4 mm
- net +3V3: track 102.2 -> 30.3 mm, vias 24 -> 0
- net DPI_SWITCH: track 0.00 -> 52.6 mm, vias 0 -> 4
- net +2V: track 51.3 -> 3.40 mm, vias 2 -> 0
- net NRST: track 90.8 -> 56.4 mm
- net NCS: track 25.5 -> 0.00 mm, vias 2 -> 0
- net MISO: track 58.4 -> 36.3 mm, vias 4 -> 2
- net USBDM: track 88.6 -> 69.5 mm, vias 4 -> 0
- net MOSI: track 42.4 -> 23.3 mm, vias 4 -> 2
- net USBDP: track 88.7 -> 70.5 mm, vias 4 -> 0
- net SWDIO: track 24.3 -> 10.1 mm
- net LEFT_CLICK: track 13.7 -> 0.00 mm
- net MIDDLE_CLICK: track 12.9 -> 0.00 mm
- net RIGHT_CLICK: track 12.7 -> 0.00 mm
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